File: Hardware/Qwiic Glove.brd (EAGLE design)
At the start: 25.4 x 36.8 mm, 24 parts, among them U4 LMV358

Commit message: updated board to sfe standards
Parts:
- added D1: RED, SparkFun-LED:LED-0603
- added R5: 1k, SparkFun-Resistors:0603
- added U$10, U$9: (no value), Labels-0_04:SCL
- added U$2: (no value), Labels-0_04:GND
- added U$5, U$6: (no value), Labels-0_04:VCC
- added U$7, U$8: (no value), Labels-0_04:SDA
- added U1: ADS1015, SparkFun-IC-Conversion:MSOP10
- J3, J4: device SparkFun-Connectors:1X02_NO_SILK -> SparkFun-Connectors:1X02
- U$1: value ADS101X-ADC_TO_I2CADS101X -> (none); device Andy:MSOP-10-GNDPAD -> Labels-0_04:GND
- moved U$1 13.9 mm to (5.08, 2.03), turned to 90 degrees
- moved C1 1.27 mm to (2.16, 6.99)
Connections:
- new net N$2: D1.C, R5.2
- net A0: now also U1.4; no longer U$1.4
- net A1: now also U1.5; no longer U$1.5
- net GND: now also R5.1, U1.3; no longer U$1.3
- net N$1: now also U1.1; no longer U$1.1
- net SCL: now also U1.10; no longer U$1.10
- net SDA: now also U1.9; no longer U$1.9
- net VCC: now also D1.A, U1.8; no longer U$1.8
Routing:
- net N$2: track 0.00 -> 10.5 mm, vias 0 -> 2
- net VCC: track 84.5 -> 85.6 mm

Commit message: PWR label
Parts:
- added U$11: (no value), Labels-0_04:(PWR)
- U$5, U$6: device Labels-0_04:VCC -> Labels-0_04:3.3V
- moved C1 21.1 mm to (23.2, 6.35), turned to 180 degrees
Changed lines of the file:
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@@
 <layer number="20" name="Dimension" color="15" fill="1" visible="yes" active="yes"/>
 <layer number="21" name="tPlace" color="16" fill="1" visible="yes" active="yes"/>
-<layer number="22" name="bPlace" color="14" fill="1" visible="no" active="yes"/>
+<layer number="22" name="bPlace" color="14" fill="1" visible="yes" active="yes"/>
 <layer number="23" name="tOrigins" color="15" fill="1" visible="yes" active="yes"/>
-<layer number="24" name="bOrigins" color="15" fill="1" visible="no" active="yes"/>
+<layer number="24" name="bOrigins" color="15" fill="1" visible="yes" active="yes"/>
 <layer number="25" name="tNames" color="7" fill="1" visible="yes" active="yes"/>
 <layer number="26" name="bNames" color="7" fill="1" visible="no" active="yes"/>
@@
 <layer number="37" name="tTest" color="7" fill="1" visible="no" active="yes"/>
 <layer number="38" name="bTest" color="7" fill="1" visible="no" active="yes"/>
-<layer number="39" name="tKeepout" color="4" fill="11" visible="no" active="yes"/>
-<layer number="40" name="bKeepout" color="1" fill="11" visible="no" active="yes"/>
+<layer number="39" name="tKeepout" color="4" fill="11" visible="yes" active="yes"/>
+<layer number="40" name="bKeepout" color="1" fill="11" visible="yes" active="yes"/>
 <layer number="41" name="tRestrict" color="4" fill="10" visible="no" active="yes"/>
 <layer number="42" name="bRestrict" color="1" fill="10" visible="no" active="yes"/>
@@
 <attribute name="PROD_ID" value="CONN-13694" x="12.7" y="20.32" size="1.778" layer="27" rot="R180" display="off"/>
 </element>
-<element name="C1" library="SparkFun-Capacitors" package="0603" value="0.1uF" x="2.159" y="6.985">
-<attribute name="PROD_ID" value="CAP-00810" x="2.159" y="6.985" size="1.778" layer="27" display="off"/>
+<element name="C1" library="SparkFun-Capacitors" package="0603" value="0.1uF" x="23.241" y="6.35" rot="R180">
+<attribute name="PROD_ID" value="CAP-00810" x="23.241" y="6.35" size="1.778" layer="27" rot="R180" display="off"/>
 </element>
 <element name="R1" library="SparkFun-Resistors" package="0603" value="4.7k" x="17.78" y="22.86" rot="R270">
@@
 <element name="U$1" library="Labels-0_04" package="GND" value="" x="5.08" y="2.032" rot="R90"/>
 <element name="U$2" library="Labels-0_04" package="GND" value="" x="5.08" y="2.032" rot="MR90"/>
-<element name="U$5" library="Labels-0_04" package="VCC" value="" x="7.62" y="2.032" rot="R90"/>
-<element name="U$6" library="Labels-0_04" package="VCC" value="" x="7.62" y="2.032" rot="MR90"/>
+<element name="U$5" library="Labels-0_04" package="3.3V" value="" x="7.62" y="2.032" rot="R90"/>
+<element name="U$6" library="Labels-0_04" package="3.3V" value="" x="7.62" y="2.032" rot="MR90"/>
 <element name="U$7" library="Labels-0_04" package="SDA" value="" x="17.78" y="2.032" rot="R90"/>
 <element name="U$8" library="Labels-0_04" package="SDA" value="" x="17.78" y="2.032" rot="MR90"/>
@@
 <attribute name="PROD_ID" value="RES-07856" x="2.159" y="2.54" size="1.778" layer="27" display="off"/>
 </element>
+<element name="U$11" library="Labels-0_04" package="(PWR)" value="" x="0.254" y="7.366"/>
 </elements>
 <signals>
@@
 <wire x1="8.89" y1="3.937" x2="9.017" y2="3.81" width="0.2032" layer="1"/>
 <wire x1="18.288" y1="3.81" x2="17.78" y2="3.81" width="0.2032" layer="1"/>
-<wire x1="22.86" y1="3.81" x2="24.13" y2="5.08" width="0.4064" layer="1"/>
-<wire x1="24.13" y1="5.08" x2="24.13" y2="7.874" width="0.4064" layer="1"/>
 <contactref element="JP3" pad="1"/>
 <wire x1="24.13" y1="7.874" x2="24.13" y2="12.065" width="0.4064" layer="1"/>
@@
 <wire x1="20.066" y1="8.89" x2="19.195" y2="8.89" width="0.2032" layer="1"/>
 <wire x1="1.27" y1="4.572" x2="1.27" y2="5.676" width="0.4064" layer="1"/>
-<wire x1="1.309" y1="6.985" x2="1.309" y2="12.026" width="0.4064" layer="1"/>
 <wire x1="1.309" y1="12.026" x2="1.27" y2="12.065" width="0.4064" layer="1"/>
 <contactref element="D1" pad="A"/>
-<wire x1="1.309" y1="6.985" x2="1.309" y2="5.488" width="0.4064" layer="1"/>
+<wire x1="24.13" y1="7.874" x2="24.13" y2="6.35" width="0.4064" layer="1"/>
+<wire x1="24.091" y1="5.041" x2="24.091" y2="6.35" width="0.4064" layer="1"/>
+<wire x1="24.091" y1="5.041" x2="22.86" y2="3.81" width="0.4064" layer="1"/>
+<wire x1="1.309" y1="12.026" x2="1.309" y2="5.488" width="0.4064" layer="1"/>
 <wire x1="1.309" y1="5.488" x2="1.282" y2="5.461" width="0.4064" layer="1"/>
-<wire x1="1.27" y1="5.676" x2="1.309" y2="5.488" width="0" layer="19" extent="1-1"/>
+<wire x1="24.091" y1="6.35" x2="24.13" y2="6.35" width="0" layer="19" extent="1-1"/>
+<wire x1="1.309" y1="5.488" x2="1.27" y2="5.676" width="0" layer="19" extent="1-1"/>
 </signal>
 <signal name="GND">
@@
 <contactref element="J2" pad="1"/>
 <via x="15.621" y="11.811" extent="1-16" drill="0.381"/>
-<via x="2.54" y="8.128" extent="1-16" drill="0.381"/>
+<via x="2.54" y="8.636" extent="1-16" drill="0.381"/>
 <via x="1.27" y="17.78" extent="1-16" drill="0.381"/>
 <via x="21.209" y="17.78" extent="1-16" drill="0.381"/>
@@
 <wire x1="3.048" y1="1.27" x2="3.048" y2="2.501" width="0.2032" layer="1"/>
 <wire x1="3.048" y1="2.501" x2="3.009" y2="2.54" width="0.2032" layer="1"/>
-<wire x1="3.036" y1="5.461" x2="4.064" y2="5.461" width="0.2032" layer="1"/>
-<wire x1="4.064" y1="5.461" x2="4.445" y2="5.842" width="0.2032" layer="1"/>
-<wire x1="4.445" y1="5.842" x2="4.445" y2="7.112" width="0.2032" layer="1"/>
-<wire x1="4.445" y1="7.112" x2="4.445" y2="2.667" width="0.2032" layer="16"/>
-<wire x1="4.445" y1="2.667" x2="3.048" y2="1.27" width="0.2032" layer="16"/>
 <via x="3.048" y="1.27" extent="1-16" drill="0.381"/>
-<via x="4.445" y="7.112" extent="1-16" drill="0.381"/>
+<via x="3.937" y="7.493" extent="1-16" drill="0.381"/>
+<wire x1="3.036" y1="5.461" x2="3.036" y2="6.592" width="0.2032" layer="1"/>
+<wire x1="3.036" y1="6.592" x2="3.937" y2="7.493" width="0.2032" layer="1"/>
+<wire x1="3.937" y1="7.493" x2="3.937" y2="2.159" width="0.2032" layer="16"/>
+<wire x1="3.937" y1="2.159" x2="3.048" y2="1.27" width="0.2032" layer="16"/>
 </signal>
 </signals>

Commit message: post checklist changes
Parts:
- removed U$3, U$4: FLEX_SENSOR, Andy:FLEX_SENSOR
- added R6, R7: FLEX_SENSOR-4.5", SparkFun-Resistors:FLEX_SENSOR
- moved C1 46.5 mm to (-23.2, 6.35), flipped to the bottom
- moved JP2 44.5 mm to (-22.2, 22.9), flipped to the top
- moved JP3 44.5 mm to (-22.2, 20.3), flipped to the top
- moved LOGO3 44.2 mm to (-21.8, 0.38), flipped to the bottom
- moved U$10 40.6 mm to (-20.3, 2.03), flipped to the top
- moved U$9 40.6 mm to (-20.3, 2.03), flipped to the bottom
- moved LOGO1 37.1 mm to (-18.5, 15.2), flipped to the top
- moved R4 36.8 mm to (-18.4, 13.3), flipped to the bottom
- moved J3 35.6 mm to (-17.8, 1.27), flipped to the bottom
- moved R1 35.6 mm to (-17.8, 22.9), flipped to the bottom
- moved U$7 35.6 mm to (-17.8, 2.03), flipped to the bottom
- moved U$8 35.6 mm to (-17.8, 2.03), flipped to the top
- moved U1 34.3 mm to (-17.1, 8.89), flipped to the bottom
- moved J1 25.4 mm to (-12.7, 20.3), flipped to the bottom
- moved J2 25.4 mm to (-12.7, 5.08), flipped to the bottom
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Connections:
- net N$3: now also R7.P$1; no longer U$3.P$1
- net N$4: now also R6.P$1; no longer U$4.P$1
- net VCC: now also R6.P$2, R7.P$2; no longer U$3.P$2, U$4.P$2
Routing:
- net VCC: track 85.6 -> 86.2 mm
Other:
- board text added: "Units in Inches"

Commit message: post review changes
Parts:
- added TP1, TP2: TEST-POINT3, SparkFun-Connectors:PAD.03X.03
- added U$12: (no value), buzzard_labels (3):SDA0
- added U$13: (no value), buzzard_labels (4):SCL2
- added U$14: (no value), buzzard_labels (4):QWIIC_GLOVE1
- added U$15: (no value), Labels:I2C-()
- added U$3: (no value), Labels:3V3-TEXT
- added U$4: (no value), Labels:GND-TEXT-03
- JP2: value JUMPER-SMT_3_1-NC_PASTE_NO-SILK -> JUMPER-SMT_3_1-NC_TRACE_NO-SILK; device SparkFun-Jumpers:SMT-JUMPER_3_1-NC_PASTE_NO-SILK -> SparkFun-Jumpers:SMT-JUMPER_3_1-NC_TRACE_NO-SILK
- JP3: value JUMPER-SMT_3_NO_NO-SILK -> JUMPER-SMT_3_NO_NO_SILK; device SparkFun-Jumpers:SMT-JUMPER_3_NO_NO-SILK -> SparkFun-Jumpers:SMT-JUMPER_3_0-NO_TRACE_NO-SILK
- moved C1 46.5 mm to (23.2, 6.35), flipped to the top
- moved R6 45.7 mm to (22.9, 12.2), flipped to the top
- moved JP2 44.5 mm to (22.2, 22.9), flipped to the bottom
- moved JP3 44.5 mm to (22.2, 20.3), flipped to the bottom
- moved FD1 43.7 mm to (21.8, 5.08), flipped to the top
- moved FD2 43.7 mm to (21.8, 5.08), flipped to the bottom
- moved LOGO3 43.7 mm to (21.8, 0.38), flipped to the top
- moved U$10 40.6 mm to (20.3, 2.03), flipped to the bottom
- moved U$9 40.6 mm to (20.3, 2.03), flipped to the top
- moved LOGO1 37.1 mm to (18.5, 15.2), flipped to the bottom
- moved R4 36.8 mm to (18.4, 13.3), flipped to the top
- moved J3 35.6 mm to (17.8, 1.27), flipped to the top
- moved R1 35.6 mm to (17.8, 22.9), flipped to the top
- moved U$7 35.6 mm to (17.8, 2.03), flipped to the top
- moved U$8 35.6 mm to (17.8, 2.03), flipped to the bottom
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Connections:
- net N$3: now also R7.P$2, TP2.P$1; no longer R7.P$1
- net N$4: now also TP1.P$1
- net VCC: now also R7.P$1; no longer R7.P$2
Routing:
- net N$3: track 4.25 -> 8.32 mm, vias 0 -> 1
- net N$4: track 13.9 -> 16.4 mm, vias 0 -> 1
Other:
- board text added: "v10"
- board text removed: "GND"
- board text removed: "I2C"
- board text removed: "Qwiic Glove"
- board text removed: "SCL"
- board text removed: "SDA"
- board text removed: "V04"
- board text removed: "VCC"
