File: Hardware/Qwiic Glove.sch (EAGLE design)
At the start: 26 parts, among them U1 ADS1015, U4 LMV358

Commit message: post review changes
Parts:
- added TP1, TP2: TEST-POINT3, SparkFun-Connectors:TEST-POINT3
- JP2: value JUMPER-SMT_3_1-NC_PASTE_NO-SILK -> JUMPER-SMT_3_1-NC_TRACE_NO-SILK; device SparkFun-Jumpers:JUMPER-SMT_3_1-NC_PASTE_NO-SILK -> SparkFun-Jumpers:JUMPER-SMT_3_1-NC_TRACE_NO-SILK
- JP3: value JUMPER-SMT_3_NO_NO-SILK -> JUMPER-SMT_3_NO_NO_SILK; device SparkFun-Jumpers:JUMPER-SMT_3_NO_NO-SILK -> SparkFun-Jumpers:JUMPER-SMT_3_NO_NO_SILK
Connections:
- net N$3: now also R7.2, TP2.1; no longer R7.1
- net N$4: now also TP1.1
- net VCC: now also R7.1; no longer R7.2
Other:
- note added: "0x48"
- note added: "0x49"
- note added: "0x4A"
- note added: "0x4B"
- note added: "v10"
- note removed: "0x90"
- note removed: "0x91"
- note removed: "0x92"
- note removed: "0x93"
- note removed: "V04"
- moved on the sheet: R7
Changed lines of the file:
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@@
 <part name="SUPPLY7" library="SparkFun-PowerSymbols" deviceset="VCC" device=""/>
 <part name="J2" library="SparkFun-Connectors" deviceset="QWIIC_CONNECTOR" device="JS-1MM"/>
-<part name="JP2" library="SparkFun-Jumpers" deviceset="JUMPER-SMT_3_1-NC_PASTE" device="_NO-SILK"/>
+<part name="JP2" library="SparkFun-Jumpers" deviceset="JUMPER-SMT_3_1-NC_TRACE" device="_NO-SILK"/>
 <part name="SUPPLY8" library="SparkFun-PowerSymbols" deviceset="VCC" device=""/>
 <part name="GND7" library="SparkFun-PowerSymbols" deviceset="GND" device=""/>
-<part name="JP3" library="SparkFun-Jumpers" deviceset="JUMPER-SMT_3_NO" device="_NO-SILK"/>
+<part name="JP3" library="SparkFun-Jumpers" deviceset="JUMPER-SMT_3_NO" device="_NO_SILK" value="JUMPER-SMT_3_NO_NO_SILK"/>
 <part name="LOGO1" library="SparkFun-Aesthetics" deviceset="SFE_LOGO_NAME_FLAME" device=".1_INCH"/>
 <part name="LOGO2" library="SparkFun-Aesthetics" deviceset="OSHW-LOGO" device="S"/>
@@
 <part name="R6" library="SparkFun-Resistors" deviceset="FLEX_SENSOR" device="-4.5&quot;"/>
 <part name="R7" library="SparkFun-Resistors" deviceset="FLEX_SENSOR" device="-4.5&quot;"/>
+<part name="TP1" library="SparkFun-Connectors" deviceset="TEST-POINT" device="3"/>
+<part name="TP2" library="SparkFun-Connectors" deviceset="TEST-POINT" device="3"/>
 </parts>
 <sheets>
 <sheet>
 <plain>
-<text x="236.22" y="7.62" size="2.54" layer="94" font="vector">V04</text>
+<text x="236.22" y="7.62" size="2.54" layer="94" font="vector">v10</text>
 <wire x1="147.32" y1="35.56" x2="147.32" y2="185.42" width="0.2032" layer="97" style="longdash"/>
 <wire x1="147.32" y1="35.56" x2="0" y2="35.56" width="0.2032" layer="97" style="longdash"/>
@@
 <wire x1="134.62" y1="127" x2="134.62" y2="114.3" width="0.2032" layer="94"/>
 <text x="139.7" y="125.73" size="1.27" layer="94" font="vector" align="center">Address</text>
-<text x="139.7" y="123.19" size="1.27" layer="94" font="vector" align="center">0x90</text>
-<text x="139.7" y="120.65" size="1.27" layer="94" font="vector" align="center">0x91</text>
-<text x="139.7" y="118.11" size="1.27" layer="94" font="vector" align="center">0x92</text>
-<text x="139.7" y="115.57" size="1.27" layer="94" font="vector" align="center">0x93</text>
+<text x="139.7" y="123.19" size="1.27" layer="94" font="vector" align="center">0x48</text>
+<text x="139.7" y="120.65" size="1.27" layer="94" font="vector" align="center">0x49</text>
+<text x="139.7" y="118.11" size="1.27" layer="94" font="vector" align="center">0x4A</text>
+<text x="139.7" y="115.57" size="1.27" layer="94" font="vector" align="center">0x4B</text>
 <text x="132.08" y="123.19" size="1.27" layer="94" font="vector" align="center">GND</text>
 <text x="132.08" y="120.65" size="1.27" layer="94" font="vector" align="center">VCC</text>
@@
 <attribute name="VALUE" x="156.464" y="127" size="1.778" layer="96" font="vector" rot="R90" align="top-center"/>
 </instance>
-<instance part="R7" gate="G$1" x="193.04" y="121.92" smashed="yes" rot="R90">
-<attribute name="NAME" x="191.516" y="121.92" size="1.778" layer="95" font="vector" rot="R90" align="bottom-center"/>
-<attribute name="VALUE" x="194.564" y="127" size="1.778" layer="96" font="vector" rot="R90" align="top-center"/>
+<instance part="R7" gate="G$1" x="193.04" y="121.92" smashed="yes" rot="R270">
+<attribute name="NAME" x="194.564" y="121.92" size="1.778" layer="95" font="vector" rot="R270" align="bottom-center"/>
+<attribute name="VALUE" x="191.516" y="116.84" size="1.778" layer="96" font="vector" rot="R270" align="top-center"/>
+</instance>
+<instance part="TP1" gate="G$1" x="160.02" y="111.76" smashed="yes" rot="R270">
+<attribute name="NAME" x="162.56" y="114.3" size="1.778" layer="95" font="vector" rot="R270"/>
+</instance>
+<instance part="TP2" gate="G$1" x="198.12" y="111.76" smashed="yes" rot="R270">
+<attribute name="NAME" x="200.66" y="114.3" size="1.778" layer="95" font="vector" rot="R270"/>
 </instance>
 </instances>
@@
 <net name="VCC" class="0">
 <segment>
-<pinref part="SUPPLY3" gate="G$1" pin="VCC"/>
-<wire x1="193.04" y1="129.54" x2="193.04" y2="127" width="0.1524" layer="91"/>
-<pinref part="R7" gate="G$1" pin="2"/>
-</segment>
-<segment>
 <pinref part="SUPPLY4" gate="G$1" pin="VCC"/>
 <wire x1="154.94" y1="129.54" x2="154.94" y2="127" width="0.1524" layer="91"/>
@@
 <wire x1="30.48" y1="81.28" x2="30.48" y2="78.74" width="0.1524" layer="91"/>
 </segment>
+<segment>
+<pinref part="R7" gate="G$1" pin="1"/>
+<pinref part="SUPPLY3" gate="G$1" pin="VCC"/>
+<wire x1="193.04" y1="127" x2="193.04" y2="129.54" width="0.1524" layer="91"/>
+</segment>
 </net>
 <net name="GND" class="0">
@@
 <net name="N$3" class="0">
 <segment>
-<wire x1="200.66" y1="114.3" x2="193.04" y2="114.3" width="0.1524" layer="91"/>
-<wire x1="193.04" y1="114.3" x2="193.04" y2="116.84" width="0.1524" layer="91"/>
+<wire x1="200.66" y1="114.3" x2="198.12" y2="114.3" width="0.1524" layer="91"/>
 <pinref part="R3" gate="G$1" pin="2"/>
+<wire x1="198.12" y1="114.3" x2="193.04" y2="114.3" width="0.1524" layer="91"/>
 <wire x1="193.04" y1="114.3" x2="193.04" y2="111.76" width="0.1524" layer="91"/>
+<pinref part="U4" gate="G2" pin="+IN"/>
+<pinref part="R7" gate="G$1" pin="2"/>
+<wire x1="193.04" y1="116.84" x2="193.04" y2="114.3" width="0.1524" layer="91"/>
 <junction x="193.04" y="114.3"/>
-<pinref part="U4" gate="G2" pin="+IN"/>
-<pinref part="R7" gate="G$1" pin="1"/>
+<pinref part="TP2" gate="G$1" pin="1"/>
+<wire x1="198.12" y1="111.76" x2="198.12" y2="114.3" width="0.1524" layer="91"/>
+<junction x="198.12" y="114.3"/>
 </segment>
 </net>
@@
 <segment>
 <pinref part="U4" gate="G1" pin="+IN"/>
-<wire x1="162.56" y1="114.3" x2="154.94" y2="114.3" width="0.1524" layer="91"/>
+<wire x1="162.56" y1="114.3" x2="160.02" y2="114.3" width="0.1524" layer="91"/>
+<wire x1="160.02" y1="114.3" x2="154.94" y2="114.3" width="0.1524" layer="91"/>
 <wire x1="154.94" y1="114.3" x2="154.94" y2="116.84" width="0.1524" layer="91"/>
 <pinref part="R4" gate="G$1" pin="2"/>
@@
 <junction x="154.94" y="114.3"/>
 <pinref part="R6" gate="G$1" pin="1"/>
-</segment>
-</net>
+<pinref part="TP1" gate="G$1" pin="1"/>
+<wire x1="160.02" y1="111.76" x2="160.02" y2="114.3" width="0.1524" layer="91"/>
+<junction x="160.02" y="114.3"/>
+</segment>
+</net>
