File: Hardware/Qwiic Flex Glove Controller.sch (EAGLE design)
At the start: 28 parts, among them U1 ADS1015, U4 LMV358

Commit message: changed to Trace Jumper
Parts:
- JP1: value JUMPER-SMT_3_2-NC_PASTE_NO-SILK -> JUMPER-SMT_3_2-NC_TRACE_NO-SILK; device SparkFun-Jumpers:JUMPER-SMT_3_2-NC_PASTE_NO-SILK -> SparkFun-Jumpers:JUMPER-SMT_3_2-NC_TRACE_NO-SILK
Changed lines of the file:
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@@
 <part name="R1" library="SparkFun-Resistors" deviceset="4.7KOHM" device="-0603-1/10W-1%" value="4.7k"/>
 <part name="R2" library="SparkFun-Resistors" deviceset="4.7KOHM" device="-0603-1/10W-1%" value="4.7k"/>
-<part name="JP1" library="SparkFun-Jumpers" deviceset="JUMPER-SMT_3_2-NC_PASTE" device="_NO-SILK"/>
+<part name="JP1" library="SparkFun-Jumpers" deviceset="JUMPER-SMT_3_2-NC_TRACE" device="_NO-SILK"/>
 <part name="SUPPLY2" library="SparkFun-PowerSymbols" deviceset="VCC" device=""/>
 <part name="GND2" library="SparkFun-PowerSymbols" deviceset="GND" device=""/>
